Commit message: wip

File: tracftec_description/urdf/mid360.urdf.xacro (robot description, xacro)
@@ -23,10 +23,10 @@
 			<visual>
 				<geometry>
-					<mesh filename="file://$(find iplow_description)/meshes/mid360.stl"/>
+					<mesh filename="file://$(find trafctec_description)/meshes/mid360.stl"/>
 				</geometry>
 			</visual>
 			<!-- <collision> -->
 			<!-- 	<geometry> -->
-			<!-- 		<mesh filename="file://$(find iplow_description)/meshes/mid360.stl"/> -->
+			<!-- 		<mesh filename="file://$(find trafctec_description)/meshes/mid360.stl"/> -->
 			<!-- 	</geometry> -->
 			<!-- </collision> -->

File: tracftec_description/urdf/right_caster.urdf.xacro (robot description, xacro)
@@ -13,10 +13,10 @@
 			<visual>
 				<geometry>
-					<mesh filename="file://$(find trafctec_description)/meshes/right_caster_pivot.stl"/>
+					<mesh filename="file://$(find tracftec_description)/meshes/right_caster_pivot.stl"/>
 				</geometry>
 			</visual>
 			<collision>
 				<geometry>
-					<mesh filename="file://$(find trafctec_description)/meshes/right_caster_pivot.stl"/>
+					<mesh filename="file://$(find tracftec_description)/meshes/right_caster_pivot.stl"/>
 				</geometry>
 			</collision>
@@ -32,10 +32,10 @@
 			<visual>
 				<geometry>
-					<mesh filename="file://$(find trafctec_description)/meshes/right_caster_wheel.stl"/>
+					<mesh filename="file://$(find tracftec_description)/meshes/right_caster_wheel.stl"/>
 				</geometry>
 			</visual>
 			<collision>
 				<geometry>
-					<mesh filename="file://$(find trafctec_description)/meshes/right_caster_wheel.stl"/>
+					<mesh filename="file://$(find tracftec_description)/meshes/right_caster_wheel.stl"/>
 				</geometry>
 			</collision>

File: tracftec_description/urdf/right_wheel.urdf.xacro (robot description, xacro)
@@ -13,10 +13,10 @@
 			<visual>
 				<geometry>
-					<mesh filename="file://$(find trafctec_description)/meshes/right_wheel.stl"/>
+					<mesh filename="file://$(find tracftec_description)/meshes/right_wheel.stl"/>
 				</geometry>
 			</visual>
 			<collision>
 				<geometry>
-					<mesh filename="file://$(find trafctec_description)/meshes/right_wheel.stl"/>
+					<mesh filename="file://$(find tracftec_description)/meshes/right_wheel.stl"/>
 				</geometry>
 			</collision>

File: tracftec_description/urdf/tracftec.urdf.xacro (robot description, xacro)
@@ -1,7 +1,7 @@
 <?xml version="1.0"?>
-<robot xmlns:xacro="http://www.ros.org/wiki/xacro" name="iplow">
+<robot xmlns:xacro="http://www.ros.org/wiki/xacro" name="tracftec">
 	<xacro:arg name="simulation" default="true"/>
 	<xacro:arg name="mid360" default="true"/>
-  <xacro:include filename="trafctec_core.urdf.xacro"/>
+  <xacro:include filename="tracftec_core.urdf.xacro"/>
   <xacro:include filename="ros2_control.urdf.xacro"/>
   <xacro:include filename="ground_truth.urdf.xacro"/>
