Commit message: wip

File: tracftec_description/urdf/left_caster.urdf.xacro (robot description, xacro)
@@ -13,10 +13,10 @@
 			<visual>
 				<geometry>
-					<mesh filename="file://$(find trafctec_description)/meshes/left_caster_pivot.stl"/>
+					<mesh filename="file://$(find tracftec_description)/meshes/left_caster_pivot.stl"/>
 				</geometry>
 			</visual>
 			<collision>
 				<geometry>
-					<mesh filename="file://$(find trafctec_description)/meshes/left_caster_pivot.stl"/>
+					<mesh filename="file://$(find tracftec_description)/meshes/left_caster_pivot.stl"/>
 				</geometry>
 			</collision>
@@ -32,10 +32,10 @@
 			<visual>
 				<geometry>
-					<mesh filename="file://$(find trafctec_description)/meshes/left_caster_wheel.stl"/>
+					<mesh filename="file://$(find tracftec_description)/meshes/left_caster_wheel.stl"/>
 				</geometry>
 			</visual>
 			<collision>
 				<geometry>
-					<mesh filename="file://$(find trafctec_description)/meshes/left_caster_wheel.stl"/>
+					<mesh filename="file://$(find tracftec_description)/meshes/left_caster_wheel.stl"/>
 				</geometry>
 			</collision>

File: tracftec_description/urdf/left_wheel.urdf.xacro (robot description, xacro)
@@ -13,10 +13,10 @@
 			<visual>
 				<geometry>
-					<mesh filename="file://$(find trafctec_description)/meshes/left_wheel.stl"/>
+					<mesh filename="file://$(find tracftec_description)/meshes/left_wheel.stl"/>
 				</geometry>
 			</visual>
 			<collision>
 				<geometry>
-					<mesh filename="file://$(find trafctec_description)/meshes/left_wheel.stl"/>
+					<mesh filename="file://$(find tracftec_description)/meshes/left_wheel.stl"/>
 				</geometry>
 			</collision>

File: tracftec_description/urdf/mid360.urdf.xacro (robot description, xacro)
@@ -23,10 +23,10 @@
 			<visual>
 				<geometry>
-					<mesh filename="file://$(find trafctec_description)/meshes/mid360.stl"/>
+					<mesh filename="file://$(find tracftec_description)/meshes/mid360.stl"/>
 				</geometry>
 			</visual>
 			<!-- <collision> -->
 			<!-- 	<geometry> -->
-			<!-- 		<mesh filename="file://$(find trafctec_description)/meshes/mid360.stl"/> -->
+			<!-- 		<mesh filename="file://$(find tracftec_description)/meshes/mid360.stl"/> -->
 			<!-- 	</geometry> -->
 			<!-- </collision> -->

File: tracftec_description/urdf/ros2_control.urdf.xacro (robot description, xacro)
@@ -44,5 +44,5 @@
     <gazebo>
       <plugin name="gazebo_ros2_control" filename="libgazebo_ros2_control.so">
-        <parameters>$(find trafctec_description)/config/gazebo_ros2_control.yaml</parameters>
+        <parameters>$(find tracftec_description)/config/gazebo_ros2_control.yaml</parameters>
       </plugin>
     </gazebo>
